Commit message: cherrypicking stuff after pulling from sitl_gazebo

File: models/rotors_description/urdf/multirotor_base.xacro (robot description, xacro)
@@ -94,5 +94,5 @@
         <geometry>
           <!-- <cylinder length="0.005" radius="${radius_rotor}"/> --> <!-- [m] -->
-          <!-- <mesh filename="package://rotors_description/meshes/propeller_${direction}.dae" -->
+          <!-- <mesh filename="package://rotors_description/meshes/${mesh}_${direction}.stl" USED FOR TYPHOON-->
           <mesh filename="package://rotors_description/meshes/${mesh}_${direction}.dae"
             scale="${mesh_scale}" />
